File: kicad/pcb/BitterDev.kicad_sch (KiCad schematic)
At the start: 19 parts, among them U1 BL24C256A-SFRC, U2 JOKER MCU, X1 ARM JTAG, Y1 7325-0800A2010-00

Commit message: Board finished (???)
Parts:
- removed C1, C10, C2, C3, C4: 100n, Capacitor_SMD:C_0402_1005Metric, symbol Device:C_Small
- removed C11: 4.7u, Capacitor_SMD:C_0402_1005Metric, symbol Device:C_Small
- removed C5: 10u, acheron_Components:CP_EIA-3216-10_Kemet-I_Pad1.58x1.35mm_HandSolder, symbol Device:CP1
- removed C6: 1u, Capacitor_SMD:C_0402_1005Metric, symbol Device:C_Small
- removed C7: 10n, Capacitor_SMD:C_0402_1005Metric, symbol Device:C_Small
- removed C8, C9: 16p, Capacitor_SMD:C_0402_1005Metric, symbol Device:C_Small
- removed R2: 4.7k, Resistor_SMD:R_0402_1005Metric, symbol Device:R_Small
- removed R3: 10k, Resistor_SMD:R_0805_2012Metric, symbol Device:R_Small
- removed R4: 1.5k, Resistor_SMD:R_0402_1005Metric, symbol Device:R_Small
- removed U1: BL24C256A-SFRC, acheron_Components:TSSOP-8_4.4x3mm_P0.65mm, symbol Memory_EEPROM:24LC256
- removed U2: JOKER MCU, acheron_Components:STM_UFQFPN-48_LQFP-48-1EP_7x7mm_P0.5mm_HandSoldering_ThermalReliefs, symbol acheron_Symbols:STM32F411-48
- removed X1: ARM JTAG, acheron_Connectors:PinHeader_2x5_P2.54mm_Vertical_Staggered, symbol Connector_Generic:Conn_02x05_Odd_Even
- removed Y1: 7325-0800A2010-00, acheron_Components:Crystal_SMD_3225-4Pin_3.2x2.5mm, symbol Device:Crystal_GND24
- added D_0, D_1, D_10, D_11, D_12, D_13, D_14, D_15, D_16, D_17, D_18, D_19, D_2, D_20, D_21, D_22, D_23, D_24, D_25, D_26, D_27, D_28, D_29, D_3, D_30, D_31, D_32, D_33, D_34, D_35, D_36, D_37, D_38, D_39, D_4, D_40, D_41, D_42, D_43, D_44, D_45, D_46, D_47, D_48, D_49, D_5, D_50, D_51, D_52, D_53, D_54, D_55, D_56, D_57, D_58, D_59, D_6, D_60, D_61, D_62, D_63, D_64, D_65, D_66, D_67, D_68, D_69, D_7, D_70, D_71, D_72, D_73, D_74, D_75, D_76, D_77, D_78, D_79, D_8, D_9: D, Keebio-Parts:Diode, symbol Device:D_Small
- added D_LED1: LED, Keebio-Parts:LED_3mm, symbol Device:LED
- added H1, H2, H3, H4: Hole, MountingHole:MountingHole_3.2mm_M3, symbol keebio:Hole
- added J1: SEN0235, BitterDev:DFRobot_EC11_Rotary_Encoder_Module, symbol BitterDev:SEN0235
- added K_0, K_1, K_10, K_11, K_12, K_13, K_14, K_15, K_16, K_17, K_18, K_19, K_2, K_20, K_21, K_22, K_23, K_24, K_25, K_27, K_28, K_29, K_3, K_30, K_31, K_32, K_33, K_34, K_35, K_36, K_37, K_38, K_39, K_4, K_41, K_42, K_43, K_44, K_45, K_46, K_47, K_48, K_49, K_5, K_50, K_51, K_52, K_53, K_54, K_55, K_56, K_57, K_58, K_59, K_6, K_60, K_61, K_62, K_63, K_64, K_65, K_66, K_67, K_68, K_69, K_7, K_70, K_71, K_73, K_75, K_76, K_77, K_78, K_79, K_8, K_9: KEYSW, Keebio-Parts:Kailh-PG1350-1u-NoLED, symbol MX_Alps_Hybrid:MX-NoLED
- added K_26, K_72, K_74: KEYSW, Keebio-Parts:Kailh-PG1350-2u-NoLED, symbol MX_Alps_Hybrid:MX-NoLED
- added K_40: KEYSW, Keebio-Parts:Kailh-PG1350-2u-Vert-NoLED, symbol MX_Alps_Hybrid:MX-NoLED
- added SW1: SW_Push, Button_Switch_THT:SW_PUSH_6mm_H4.3mm, symbol Switch:SW_Push
- added U1, U2: ProMicro, Keebio-Parts:ArduinoProMicro, symbol keebio:ProMicro
- R1: value 4.7k -> R_Small; footprint Resistor_SMD:R_0402_1005Metric -> Keebio-Parts:Resistor; Package R0402 -> (none)
Connections:
- net GND: now also D_LED1.1 (K), J1.2 (GND), SW1.2, U1.23 (GND), U1.3 (GND), U1.4 (GND), U2.23 (GND), U2.3 (GND), U2.4 (GND)
- net 3V3 renamed CAPS
- net CAPS: now also U1.13 (10/PB6)
- net SDA: no longer names the net of R1.2
- net SDA: now also D_LED1.2 (A)
- new net: D_65.2 (A), K_65.2 (ROW)
- new net: D_40.2 (A), K_40.2 (ROW)
- new net: D_24.2 (A), K_24.2 (ROW)
- new net: D_79.2 (A), K_79.2 (ROW)
- new net: D_53.2 (A), K_53.2 (ROW)
- new net: D_71.2 (A), K_71.2 (ROW)
- new net: D_75.2 (A), K_75.2 (ROW)
- new net: D_3.2 (A), K_3.2 (ROW)
- new net: D_76.2 (A), K_76.2 (ROW)
- new net: D_52.2 (A), K_52.2 (ROW)
- new net: D_50.2 (A), K_50.2 (ROW)
- new net: D_6.2 (A), K_6.2 (ROW)
- new net: D_42.2 (A), K_42.2 (ROW)
- new net: D_30.2 (A), K_30.2 (ROW)
- new net: D_60.2 (A), K_60.2 (ROW)
- new net: D_2.2 (A), K_2.2 (ROW)
- new net: D_69.2 (A), K_69.2 (ROW)
- new net: D_73.2 (A), K_73.2 (ROW)
- new net: D_29.2 (A), K_29.2 (ROW)
- new net: D_39.2 (A), K_39.2 (ROW)
- new net: D_36.2 (A), K_36.2 (ROW)
- new net: D_74.2 (A), K_74.2 (ROW)
- new net: D_35.2 (A), K_35.2 (ROW)
- new net: D_32.2 (A), K_32.2 (ROW)
- new net: D_61.2 (A), K_61.2 (ROW)
- new net: D_46.2 (A), K_46.2 (ROW)
- new net: D_8.2 (A), K_8.2 (ROW)
- new net: D_22.2 (A), K_22.2 (ROW)
- new net: D_31.2 (A), K_31.2 (ROW)
- new net: D_58.2 (A), K_58.2 (ROW)
- new net: D_62.2 (A), K_62.2 (ROW)
- new net: D_0.2 (A), K_0.2 (ROW)
- new net: D_20.2 (A), K_20.2 (ROW)
- new net: D_63.2 (A), K_63.2 (ROW)
- new net: D_15.2 (A), K_15.2 (ROW)
- new net: D_59.2 (A), K_59.2 (ROW)
- new net: D_41.2 (A), K_41.2 (ROW)
- new net: D_10.2 (A), K_10.2 (ROW)
- new net: D_37.2 (A), K_37.2 (ROW)
- new net: D_26.2 (A), K_26.2 (ROW)
- new net: D_21.2 (A), K_21.2 (ROW)
- new net: D_25.2 (A), K_25.2 (ROW)
- new net: D_64.2 (A), K_64.2 (ROW)
- new net: D_54.2 (A), K_54.2 (ROW)
- new net: D_47.2 (A), K_47.2 (ROW)
- new net: D_5.2 (A), K_5.2 (ROW)
- new net: D_4.2 (A), K_4.2 (ROW)
- new net: D_34.2 (A), K_34.2 (ROW)
- new net: D_56.2 (A), K_56.2 (ROW)
- new net: D_48.2 (A), K_48.2 (ROW)
- new net: D_19.2 (A), K_19.2 (ROW)
- new net: D_43.2 (A), K_43.2 (ROW)
- new net: D_12.2 (A), K_12.2 (ROW)
- new net: D_16.2 (A), K_16.2 (ROW)
- new net: D_33.2 (A), K_33.2 (ROW)
- new net: D_77.2 (A), K_77.2 (ROW)
- new net: D_9.2 (A), K_9.2 (ROW)
- new net: D_18.2 (A), K_18.2 (ROW)
- new net: D_51.2 (A), K_51.2 (ROW)
- new net: D_44.2 (A), K_44.2 (ROW)
- new net: D_28.2 (A), K_28.2 (ROW)
- new net: D_17.2 (A), K_17.2 (ROW)
- new net: D_14.2 (A), K_14.2 (ROW)
- new net: D_7.2 (A), K_7.2 (ROW)
- new net: D_27.2 (A), K_27.2 (ROW)
- new net: D_38.2 (A), K_38.2 (ROW)
- new net: D_57.2 (A), K_57.2 (ROW)
- new net: D_45.2 (A), K_45.2 (ROW)
- new net: D_23.2 (A), K_23.2 (ROW)
- new net: D_70.2 (A), K_70.2 (ROW)
- new net: D_68.2 (A), K_68.2 (ROW)
- new net: D_55.2 (A), K_55.2 (ROW)
- new net: D_78.2 (A), K_78.2 (ROW)
- new net: D_66.2 (A), K_66.2 (ROW)
- new net: D_49.2 (A), K_49.2 (ROW)
- new net: D_13.2 (A), K_13.2 (ROW)
- new net: D_11.2 (A), K_11.2 (ROW)
- new net: D_72.2 (A), K_72.2 (ROW)
- new net: D_67.2 (A), K_67.2 (ROW)
- new net: D_1.2 (A), K_1.2 (ROW)
- new net DATA: U1.1 (TX0/PD3), U2.1 (TX0/PD3)
- new net ENC_A: J1.3 (A), U1.5 (2/PD1)
- new net ENC_B: J1.4 (B), U1.6 (3/PD0)
- new net RST: SW1.1, U1.22 (RST), U2.22 (RST)
- new net VCC: J1.1 (VCC), U1.21 (VCC), U2.21 (VCC)
- new net col0: K_0.1 (COL), K_13.1 (COL), K_27.1 (COL), K_41.1 (COL), K_54.1 (COL), K_68.1 (COL), U1.14 (16/PB2)
- new net col1: K_14.1 (COL), K_28.1 (COL), K_42.1 (COL), K_55.1 (COL), K_69.1 (COL), U1.7 (4/PD4)
- new net col10: K_23.1 (COL), K_37.1 (COL), K_51.1 (COL), K_64.1 (COL), K_76.1 (COL), K_9.1 (COL), U2.19 (A2/PF5)
- new net col11: K_10.1 (COL), K_24.1 (COL), K_38.1 (COL), K_52.1 (COL), K_65.1 (COL), K_77.1 (COL), U2.20 (A3/PF4)
- new net col12: K_11.1 (COL), K_25.1 (COL), K_39.1 (COL), K_53.1 (COL), K_66.1 (COL), K_78.1 (COL), U2.12 (9/PB5)
- new net col13: K_12.1 (COL), K_26.1 (COL), K_40.1 (COL), K_67.1 (COL), K_79.1 (COL), U2.11 (8/PB4)
- new net col2: K_1.1 (COL), K_15.1 (COL), K_29.1 (COL), K_43.1 (COL), K_56.1 (COL), K_70.1 (COL), U1.8 (5/PC6)
- new net col3: K_16.1 (COL), K_2.1 (COL), K_30.1 (COL), K_44.1 (COL), K_57.1 (COL), K_71.1 (COL), U1.9 (6/PD7)
- new net col4: K_17.1 (COL), K_3.1 (COL), K_31.1 (COL), K_45.1 (COL), K_58.1 (COL), K_72.1 (COL), U1.10 (7/PE6)
- new net col5: K_18.1 (COL), K_32.1 (COL), K_4.1 (COL), K_46.1 (COL), K_59.1 (COL), U1.11 (8/PB4)
- new net col6: K_19.1 (COL), K_33.1 (COL), K_47.1 (COL), K_5.1 (COL), K_60.1 (COL), K_73.1 (COL), U1.12 (9/PB5)
- new net col7: K_20.1 (COL), K_34.1 (COL), K_48.1 (COL), K_6.1 (COL), K_61.1 (COL), K_74.1 (COL), U2.16 (15/PB1)
- new net col8: K_21.1 (COL), K_35.1 (COL), K_49.1 (COL), K_62.1 (COL), K_7.1 (COL), U2.17 (A0/PF7)
- new net col9: K_22.1 (COL), K_36.1 (COL), K_50.1 (COL), K_63.1 (COL), K_75.1 (COL), K_8.1 (COL), U2.18 (A1/PF6)
- new net row0a: D_0.1 (K), D_1.1 (K), D_2.1 (K), D_3.1 (K), D_4.1 (K), D_5.1 (K), U1.15 (14/PB3)
- new net row0b: D_10.1 (K), D_11.1 (K), D_12.1 (K), D_6.1 (K), D_7.1 (K), D_8.1 (K), D_9.1 (K), U2.10 (7/PE6)
- new net row1a: D_13.1 (K), D_14.1 (K), D_15.1 (K), D_16.1 (K), D_17.1 (K), D_18.1 (K), D_19.1 (K), U1.16 (15/PB1)
- new net row1b: D_20.1 (K), D_21.1 (K), D_22.1 (K), D_23.1 (K), D_24.1 (K), D_25.1 (K), D_26.1 (K), U2.9 (6/PD7)
- new net row2a: D_27.1 (K), D_28.1 (K), D_29.1 (K), D_30.1 (K), D_31.1 (K), D_32.1 (K), D_33.1 (K), U1.17 (A0/PF7)
- new net row2b: D_34.1 (K), D_35.1 (K), D_36.1 (K), D_37.1 (K), D_38.1 (K), D_39.1 (K), D_40.1 (K), U2.8 (5/PC6)
- new net row3a: D_41.1 (K), D_42.1 (K), D_43.1 (K), D_44.1 (K), D_45.1 (K), D_46.1 (K), D_47.1 (K), U1.18 (A1/PF6)
- new net row3b: D_48.1 (K), D_49.1 (K), D_50.1 (K), D_51.1 (K), D_52.1 (K), D_53.1 (K), U2.7 (4/PD4)
- new net row4a: D_54.1 (K), D_55.1 (K), D_56.1 (K), D_57.1 (K), D_58.1 (K), D_59.1 (K), D_60.1 (K), U1.19 (A2/PF5)
- new net row4b: D_61.1 (K), D_62.1 (K), D_63.1 (K), D_64.1 (K), D_65.1 (K), D_66.1 (K), D_67.1 (K), U2.6 (3/PD0)
- new net row5a: D_68.1 (K), D_69.1 (K), D_70.1 (K), D_71.1 (K), D_72.1 (K), D_73.1 (K), U1.20 (A3/PF4)
- new net row5b: D_74.1 (K), D_75.1 (K), D_76.1 (K), D_77.1 (K), D_78.1 (K), D_79.1 (K), U2.5 (2/PD1)
- no-connect marks 0 -> 8
Other:
- note removed: "(*) "Spooky pins": on STM32F4x1, pins A9 and B2 cannot be used for switch matrix: - A9 is meant to be used as a VBUS sensing. It has a undocumented internal pulldown resistor; - B2 is used as BOOT1 during bootup, so it needs an external pulldown for successful bootup; - B13 is locked by the SPI driver on the MCUs that use it for RGB drive;"
- note removed: "(**) PA9 jumper: a solderable jumper used to tie PA9 to VBUS. It is disconnected by default, hence PA9 is left floating"
- note removed: "EEPROM"
- note removed: "MCU"
- note removed: "Spooky pin (*)"
